File: pcb/main_box/main_box.kicad_sch (KiCad schematic)
At the start: 20 parts, among them J1 AudioJack4, J13 Conn_01x06, J2 AudioJack4, J3 AudioJack4, J4 AudioJack4, J5 AudioJack4, J6 AudioJack4, J7 AudioJack4, J8 AudioJack4, SW1 SW_Push, SW2 SW_Push, SW3 SW_Push, SW4 SW_Push, SW5 SW_Push, SW6 SW_Push, U1 Pico

Commit message: Mby somewhat done...
Parts:
- removed J13: Conn_01x06, Connector_JST:JST_XH_B6B-XH-A_1x06_P2.50mm_Vertical, symbol Connector_Generic:Conn_01x06
- added J9: Conn_01x06_MountingPin, symbol Connector_Generic_MountingPin:Conn_01x06_MountingPin
- SW1, SW2, SW3, SW4, SW5, SW6: footprint Button_Switch_THT:SW_PUSH_6mm -> Audio-jacks Libraries:SW_PUSH_combined_6mm
Connections:
- net +3V3: now also J9.5 (Pin_5)
- net ADC0: now also J9.2 (Pin_2)
- net ADC1: now also J9.3 (Pin_3)
- net ADC2: now also J9.4 (Pin_4)
- net GND: now also J9.6 (Pin_6), J9.MP (MountPin)
- net GPIO22: now also J9.1 (Pin_1)
- net GPIO3: now also J7.R2; no longer J7.T
- net GPIO5: now also J7.T; no longer J7.R2
Changed lines of the file:
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@@
 	(paper "A4")
 	(junction
+		(at 133.35 57.15)
+		(diameter 0)
+		(color 0 0 0 0)
+	)
+	(junction
 		(at 22.86 60.96)
 		(diameter 0)
@@
 	(wire
 		(pts
+			(xy 142.24 54.61) (xy 142.24 57.15)
+		)
+		(stroke
+			(width 0)
+			(type default)
+		)
+	)
+	(wire
+		(pts
 			(xy 233.68 82.55) (xy 233.68 85.09)
 		)
@@
 	(wire
 		(pts
+			(xy 142.24 57.15) (xy 133.35 57.15)
+		)
+		(stroke
+			(width 0)
+			(type default)
+		)
+	)
+	(wire
+		(pts
 			(xy 38.1 76.2) (xy 26.67 76.2)
 		)
@@
 	(wire
 		(pts
-			(xy 133.35 52.07) (xy 133.35 49.53)
+			(xy 133.35 59.69) (xy 133.35 57.15)
 		)
 		(stroke
@@
 	(wire
 		(pts
-			(xy 195.58 100.33) (xy 184.15 100.33)
+			(xy 195.58 105.41) (xy 184.15 105.41)
 		)
 		(stroke
@@
 	(wire
 		(pts
+			(xy 133.35 57.15) (xy 133.35 49.53)
+		)
+		(stroke
+			(width 0)
+			(type default)
+		)
+	)
+	(wire
+		(pts
 			(xy 224.79 57.15) (xy 236.22 57.15)
 		)
@@
 	(wire
 		(pts
-			(xy 184.15 105.41) (xy 195.58 105.41)
+			(xy 184.15 100.33) (xy 195.58 100.33)
 		)
 		(stroke
@@
 	)
 	(label "GPIO3"
-		(at 184.15 100.33 0)
+		(at 184.15 105.41 0)
 		(fields_autoplaced yes)
 		(effects
@@
 	)
 	(label "GPIO5"
-		(at 184.15 105.41 0)
+		(at 184.15 100.33 0)
 		(fields_autoplaced yes)
 		(effects
@@
 			)
 		)
-		(property "Footprint" "Button_Switch_THT:SW_PUSH_6mm"
+		(property "Footprint" "Audio-jacks Libraries:SW_PUSH_combined_6mm"
 			(at 205.74 52.07 0)
 			(effects
@@
 	)
 	(symbol
-		(lib_id "Connector_Generic:Conn_01x06")
-		(at 142.24 44.45 0)
-		(mirror x)
+		(lib_id "Switch:SW_Push")
+		(at 241.3 36.83 0)
 		(unit 1)
 		(exclude_from_sim no)
@@
 		(dnp no)
 		(fields_autoplaced yes)
-		(property "Reference" "J13"
-			(at 142.24 30.48 0)
+		(property "Reference" "SW5"
+			(at 241.3 29.21 0)
 			(effects
 				(font
@@
 			)
 		)
-		(property "Value" "Conn_01x06"
-			(at 142.24 33.02 0)
+		(property "Value" "SW_Push"
+			(at 241.3 31.75 0)
 			(effects
 				(font
@@
 			)
 		)
-		(property "Footprint" "Connector_JST:JST_XH_B6B-XH-A_1x06_P2.50mm_Vertical"
-			(at 142.24 44.45 0)
+		(property "Footprint" "Audio-jacks Libraries:SW_PUSH_combined_6mm"
+			(at 241.3 31.75 0)
 			(effects
 				(font
@@
 		)
 		(property "Datasheet" "~"
-			(at 142.24 44.45 0)
+			(at 241.3 31.75 0)
 			(effects
 				(font
@@
 			)
 		)
-		(property "Description" "Generic connector, single row, 01x06, script generated (kicad-library-utils/schlib/autogen/connector/)"
-			(at 142.24 44.45 0)
+		(property "Description" "Push button switch, generic, two pins"
+			(at 241.3 36.83 0)
 			(effects
 				(font
@@
 			)
 		)
-		(pin "2"
-		)
 		(pin "1"
 		)
-		(pin "3"
-		)
-		(pin "4"
-		)
-		(pin "6"
-		)
-		(pin "5"
+		(pin "2"
 		)
 		(instances
-			(project ""
+			(project "main_box"
 				(path "/9a1cce8c-db89-40d4-b1fe-9e94eaa8821d"
-					(reference "J13")
+					(reference "SW5")
 					(unit 1)
 				)
@@
 	)
 	(symbol
-		(lib_id "Switch:SW_Push")
-		(at 241.3 36.83 0)
+		(lib_id "Connector_Generic_MountingPin:Conn_01x06_MountingPin")
+		(at 142.24 41.91 0)
 		(unit 1)
 		(exclude_from_sim no)
@@
 		(on_board yes)
 		(dnp no)
-		(fields_autoplaced yes)
-		(property "Reference" "SW5"
-			(at 241.3 29.21 0)
+		(property "Reference" "J9"
+			(at 136.652 28.956 0)
 			(effects
 				(font
 					(size 1.27 1.27)
 				)
+				(justify left)
 			)
 		)
-		(property "Value" "SW_Push"
-			(at 241.3 31.75 0)
+		(property "Value" "Conn_01x06_MountingPin"
+			(at 136.652 31.496 0)
 			(effects
 				(font
 					(size 1.27 1.27)
 				)
+				(justify left)
 			)
 		)
-		(property "Footprint" "Button_Switch_THT:SW_PUSH_6mm"
-			(at 241.3 31.75 0)
+		(property "Footprint" ""
+			(at 142.24 41.91 0)
 			(effects
 				(font
@@
 		)
 		(property "Datasheet" "~"
-			(at 241.3 31.75 0)
+			(at 142.24 41.91 0)
 			(effects
 				(font
@@
 			)
 		)
-		(property "Description" "Push button switch, generic, two pins"
-			(at 241.3 36.83 0)
+		(property "Description" "Generic connectable mounting pin connector, single row, 01x06, script generated (kicad-library-utils/schlib/autogen/connector/)"
+			(at 142.24 41.91 0)
 			(effects
 				(font
@@
 		(pin "2"
 		)
+		(pin "MP"
+		)
+		(pin "6"
+		)
+		(pin "3"
+		)
+		(pin "4"
+		)
+		(pin "5"
+		)
 		(instances
-			(project "main_box"
+			(project ""
 				(path "/9a1cce8c-db89-40d4-b1fe-9e94eaa8821d"
-					(reference "SW5")
+					(reference "J9")
 					(unit 1)
 				)
@@
 			)
 		)
-		(property "Footprint" "Button_Switch_THT:SW_PUSH_6mm"
+		(property "Footprint" "Audio-jacks Libraries:SW_PUSH_combined_6mm"
 			(at 205.74 31.75 0)
 			(effects
@@
 	(symbol
 		(lib_id "power:GND")
-		(at 133.35 52.07 0)
+		(at 133.35 59.69 0)
 		(mirror y)
 		(unit 1)
@@
 		(fields_autoplaced yes)
 		(property "Reference" "#PWR028"
-			(at 133.35 58.42 0)
+			(at 133.35 66.04 0)
 			(effects
 				(font
@@
 		)
 		(property "Value" "GND"
-			(at 133.35 57.15 0)
+			(at 133.35 64.77 0)
 			(effects
 				(font
@@
 		)
 		(property "Footprint" ""
-			(at 133.35 52.07 0)
+			(at 133.35 59.69 0)
 			(effects
 				(font
@@
 		)
 		(property "Datasheet" ""
-			(at 133.35 52.07 0)
+			(at 133.35 59.69 0)
 			(effects
 				(font
@@
 		)
 		(property "Description" "Power symbol creates a global label with name \"GND\" , ground"
-			(at 133.35 52.07 0)
+			(at 133.35 59.69 0)
 			(effects
 				(font
@@
 			)
 		)
-		(property "Footprint" "Button_Switch_THT:SW_PUSH_6mm"
+		(property "Footprint" "Audio-jacks Libraries:SW_PUSH_combined_6mm"
 			(at 168.91 52.07 0)
 			(effects
@@
 			)
 		)
-		(property "Footprint" "Button_Switch_THT:SW_PUSH_6mm"
+		(property "Footprint" "Audio-jacks Libraries:SW_PUSH_combined_6mm"
 			(at 168.91 31.75 0)
 			(effects
@@
 			)
 		)
-		(property "Footprint" "Button_Switch_THT:SW_PUSH_6mm"
+		(property "Footprint" "Audio-jacks Libraries:SW_PUSH_combined_6mm"
 			(at 241.3 52.07 0)
 			(effects

Commit message: Getting there, just buttons are still small...
Parts:
- removed J1, J2, J3, J4, J5, J6, J7, J8: AudioJack4, Audio-jacks Libraries:SJ2_SJ3_combined, symbol Connector_Audio:AudioJack4
- removed J9: Conn_01x06_MountingPin, symbol Connector_Generic_MountingPin:Conn_01x06_MountingPin
- added H5, H6, H7, H8: MountingHole, MountingHole:MountingHole_3.2mm_M3, symbol Mechanical:MountingHole
- added J1, J2, J3, J4, J5, J6, J7, J8: AudioJack4_SwitchTR1, Audio-jacks Libraries:Jack_3.5_PJ31060-I_L_pads, symbol Connector_Audio:AudioJack4_SwitchTR1
- added J9: Conn_01x05_MountingPin, Audio-jacks Libraries:JST_XH_S5B_combined_1x05, symbol Connector_Generic_MountingPin:Conn_01x05_MountingPin
Connections:
- net +3V3: now also J7.R2, J8.R2, J9.4 (Pin_4)
- net ADC0: now also J8.T
- net ADC1: now also J7.R1, J7.R1N
- net ADC2: now also J8.R1
- net GND: now also J1.S, J2.S, J3.S, J4.S, J5.S, J6.S, J7.S, J8.S, J9.5 (Pin_5), J9.MP (MountPin)
- net GPIO0: now also J1.R2
- net GPIO1: now also J1.T, J1.TN
- net GPIO10: now also J4.T, J4.TN
- net GPIO11: now also J4.R1, J4.R1N
- net GPIO12: now also SW1.1; no longer SW6.1
- net GPIO13: now also SW2.1; no longer SW5.1
- net GPIO14: now also SW3.1; no longer SW4.1
- net GPIO15: now also SW4.1; no longer SW3.1
- net GPIO16: now also SW5.1, J5.R2; no longer SW2.1
- net GPIO17: now also SW6.1, J5.T, J5.TN; no longer SW1.1
- net GPIO18: now also J5.R1, J5.R1N
- net GPIO19: now also J6.R2
- net GPIO2: now also J1.R1, J1.R1N
- net GPIO20: now also J6.T, J6.TN
- net GPIO21: now also J6.R1, J6.R1N
- net GPIO22: now also J7.T, J7.TN, J9.3 (Pin_3)
- net GPIO3: now also J2.R2
- net GPIO4: now also J2.T, J2.TN
- net GPIO5: now also J2.R1, J2.R1N
- net GPIO6: now also J3.R2
- net GPIO7: now also J3.T, J3.TN
- net GPIO8: now also J3.R1, J3.R1N
- net GPIO9: now also J4.R2
- new net ADC0_N: J8.TN, J9.2 (Pin_2)
- new net ADC2_N: J8.R1N, J9.1 (Pin_1)
Other:
- note added: "A"
- note added: "B"
- note added: "HOME"
- note added: "MENU"
- note added: "X"
- note added: "Y"
- moved on the sheet: SW1, SW2, SW3, SW4, SW5, SW6

Commit message: Maybe done, but some refactoring is needed
Parts:
- removed H5, H6, H7, H8: MountingHole, MountingHole:MountingHole_3.2mm_M3, symbol Mechanical:MountingHole
- added H9: Joystick module - 4 MP, Audio-jacks Libraries:Joystick_module_lifted, symbol Audio-jacks Libraries:Joystick_module
Other:
- note added: "->"
- moved on the sheet: J9, SW1, SW2, SW3, SW4, SW5, SW6
